Commit message: Add wrist camera and teleoperator node

File: urdf/armando_body.urdf.xacro (robot description, xacro)
@@ -389,5 +389,5 @@
         </inertial>
     </link>
-    <!-- Frame di montaggio della camera (end-effector) -->
+    <!-- Frame di montaggio della camera (base frame) -->
     <joint name="camera_mount_joint" type="fixed">
         <parent link="base_link"/>

File: urdf/armando_camera.urdf.xacro (robot description, xacro)
@@ -41,3 +41,51 @@
         </sensor>
     </gazebo>
+    % Aggiunta nuova camera
+    <!-- Camera solidale alla base della pinza -->
+    <joint name="wrist_camera_joint" type="fixed">
+        <parent link="crawer_base"/>
+        <child link="wrist_camera_link"/>
+        <!-- Posizione espressa negli assi di crawer_base.
+            Rotazione: +X della camera punta verso +Y della pinza. -->
+            <!--Si colloca la camera a 4 cm lungo l'asse Z locale della pinza -->
+        <origin xyz="0.0 0.0 0.04"
+                rpy="0 -1.57079632679 0"/>
+                <!--Ci dice dove guarda fisicamente il sensore rispetto alla pinza-->
+    </joint>
+    <link name="wrist_camera_link">
+        <visual>
+            <geometry>
+                <box size="0.01 0.03 0.03"/>
+            </geometry>
+            <material name="red"/>
+        </visual>
+    </link>
+    <!-- Convenzione ottica: Z avanti, X destra, Y basso -->
+    <joint name="wrist_camera_optical_joint" type="fixed">
+        <parent link="wrist_camera_link"/>
+        <child link="wrist_camera_optical_frame"/>
+        <origin xyz="0 0 0"
+                rpy="-1.57079632679 0 -1.57079632679"/>
+    </joint>
+    <link name="wrist_camera_optical_frame"/>
+    <gazebo reference="wrist_camera_link">
+        <sensor name="wrist_camera" type="camera">
+            <camera>
+                <horizontal_fov>1.047</horizontal_fov>
+                <image>
+                    <width>640</width>
+                    <height>480</height>
+                </image>
+                <clip>
+                    <near>0.02</near>
+                    <far>5.0</far>
+                </clip>
+            </camera>
+            <always_on>1</always_on>
+            <update_rate>30</update_rate>
+            <visualize>true</visualize>
+            <topic>/wrist_camera/image</topic>
+            <gz_frame_id>wrist_camera_optical_frame</gz_frame_id>
+        </sensor>
+    </gazebo>
 </robot>
